Commit message: add inertial property to virtual links to make it compatible with gazebo

File: iai_boxy_base_2/robots/base.URDF (robot description, URDF)
Before this commit: robot base, 8 links, 7 joints
Links:
- link laser_reference_back: mass None -> 0.01
- link laser_reference_front: mass None -> 0.01
- link odom: mass None -> 0.01
- link odom_x_frame: mass None -> 0.01
- link odom_y_frame: mass None -> 0.01

File: iai_donbot_description/robots/iai_donbot.xacro (robot description, xacro)
@@ -1,6 +1,6 @@
 <?xml version="1.0"?>
 <robot xmlns:xacro="http://www.ros.org/wiki/xacro">
-  <xacro:include filename="$(find ur_description)/urdf/common.gazebo.xacro" />
-  <xacro:include filename="$(find ur_description)/urdf/ur5.urdf.xacro" />
+  <xacro:include filename="$(find iai_ur_description)/urdf/common.gazebo.xacro" />
+  <xacro:include filename="$(find iai_ur_description)/urdf/ur5.urdf.xacro" />
   <xacro:include filename="$(find iai_kms_40_description)/urdf/kms_40.urdf.xacro"/>
   <xacro:include filename="$(find iai_adapters_description)/urdf/adapter_fwa050_wsg50.urdf.xacro"/>
